File: Topographic Robot/Topographic Robot.kicad_sch (KiCad schematic)
At the start: 0 parts

Commit message: Movement + Sensors
Other:
- added sheet Movement (Movement.kicad_sch)
Changed lines of the file:
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@@
+	)
+	(sheet
+		(at 12.7 30.48)
+		(size 16.51 11.43)
+		(fields_autoplaced yes)
+		(stroke
+			(width 0.1524)
+			(type solid)
+		)
+		(fill
+			(color 0 0 0 0.0000)
+		)
+		(property "Sheetname" "Movement"
+			(at 12.7 29.7684 0)
+			(effects
+				(font
+					(size 1.27 1.27)
+				)
+				(justify left bottom)
+			)
+		)
+		(property "Sheetfile" "Movement.kicad_sch"
+			(at 12.7 42.4946 0)
+			(effects
+				(font
+					(size 1.27 1.27)
+				)
+				(justify left top)
+			)
+		)
+		(property "Field2" ""
+			(at 12.7 30.48 0)
+			(effects
+				(font
+					(size 1.27 1.27)
+				)
+				(hide yes)
+			)
+		)
+		(instances
+			(project "Topographic Robot"
+				(path "/67e33313-0ce8-4ff5-8d50-46dc6ab8d472"
+					(page "4")
+				)
+			)
+		)
 	)
 	(sheet

Commit message: THEY ARE QUAD TRISTATE BUFFERS TOOO SOOOOO I GOT 400 TRISTATE BUFFERS!!!!!
Other:
- added sheet Vision (Vision.kicad_sch)
Changed lines of the file:
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@@
+		)
+	)
+	(sheet
+		(at 38.1 33.02)
+		(size 21.59 7.62)
+		(fields_autoplaced yes)
+		(stroke
+			(width 0.1524)
+			(type solid)
+		)
+		(fill
+			(color 0 0 0 0.0000)
+		)
+		(property "Sheetname" "Vision"
+			(at 38.1 32.3084 0)
+			(effects
+				(font
+					(size 1.27 1.27)
+				)
+				(justify left bottom)
+			)
+		)
+		(property "Sheetfile" "Vision.kicad_sch"
+			(at 38.1 41.2246 0)
+			(effects
+				(font
+					(size 1.27 1.27)
+				)
+				(justify left top)
+			)
+		)
+		(instances
+			(project "Topographic Robot"
+				(path "/67e33313-0ce8-4ff5-8d50-46dc6ab8d472"
+					(page "5")
+				)
+			)
 		)
 	)
