File: Topographic Robot/Vision.kicad_sch (KiCad schematic)
At the start: 25 parts, among them U17 OV7670, U18 OV7670, U19 OV7670, U20 OV7670, U21 OV7670, U22 OV7670, U23 PCA9548A, U27 74LVC125AD, U28 74LVC125AD, U29 74LVC125AD, U30 74LVC125AD, U31 74LVC125AD, U32 74LVC125AD, U33 74LVC125AD, U34 74LVC125AD, U35 74LVC125AD, U36 74LVC125AD, U37 74LVC125AD, U38 74LVC125AD, U39 74LVC125AD, U40 74LVC125AD, U41 74LVC125AD, U42 74LVC125AD, U43 74LVC125AD, U44 74LVC125AD

Commit message: Parallel > USB ?!
Parts:
- added U24: DE10-Lite_GPIO, symbol FPGA_Terasic_Simple:DE10-Lite_GPIO
- added U25: RaspberryPi_Zero_2W, symbol MCU_RaspberryPi_Simple:RaspberryPi_Zero_2W
Connections:
- net FPGA_D0: now also U24. (GPIO_9)
- net FPGA_D1: now also U24. (GPIO_9)
- net FPGA_D2: now also U24. (GPIO_9)
- net FPGA_D3: now also U24. (GPIO_9)
- net FPGA_D4: now also U24. (GPIO_9); no longer U44. (VCC)
- net FPGA_D5: now also U24. (GPIO_9); no longer U44. (VCC)
- net FPGA_D6: now also U24. (GPIO_9); no longer U44. (VCC)
- net FPGA_D7: now also U24. (GPIO_9)
- net FPGA_E_C0: now also U24. (GPIO_9)
- net FPGA_E_C1: now also U24. (GPIO_9)
- net FPGA_E_C2: now also U24. (GPIO_9)
- net FPGA_E_C3: now also U24. (GPIO_9)
- net FPGA_E_C4: now also U24. (GPIO_9)
- net FPGA_E_C5: now also U24. (GPIO_9)
- net FPGA_HREF: now also U44. (VCC), U24. (GPIO_9)
- net FPGA_PCLK: now also U44. (VCC), U24. (GPIO_9)
- net FPGA_VSYNC: now also U44. (VCC), U24. (GPIO_9)
- net FPGA_XCLK: now also U24. (GPIO_9)
- net GND: now also U24. (GPIO_9), U25. (GPIO_9)
- new net: U24. (GPIO_9), U25. (GPIO_9) (x18)
- new net 5V: U24. (GPIO_9), U25. (GPIO_9)
- no-connect marks 16 -> 31
Other:
- note added: "Cameras"
- note added: "FPGA + MCU"
- note added: "Tristate Buffers"
- moved on the sheet: U23, U27, U28, U29, U30, U31, U32, U33, U34, U35, U36, U37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
