File: 6V_Power_Line.kicad_sch (KiCad schematic)
At the start: 26 parts, among them Q13 CSD19502Q5B, Q7 CSD19502Q5B, U9 LM25145RGYR

Commit message: 20V line PCB v1
Parts:
- removed C100, C101: 10u, Capacitor_SMD:C_0805_2012Metric_Pad1.18x1.45mm_HandSolder, symbol Device:C_Small
- removed C91: 4.7u, Capacitor_SMD:C_0805_2012Metric_Pad1.18x1.45mm_HandSolder, symbol Device:C_Small
- removed C92: 56n, Capacitor_SMD:C_0805_2012Metric_Pad1.18x1.45mm_HandSolder, symbol Device:C_Small
- removed C93: 2.2u, Capacitor_SMD:C_0805_2012Metric_Pad1.18x1.45mm_HandSolder, symbol Device:C_Small
- removed C94, C96: 100n, Capacitor_SMD:C_0805_2012Metric_Pad1.18x1.45mm_HandSolder, symbol Device:C_Small
- removed C95: 10p, Capacitor_SMD:C_0805_2012Metric_Pad1.18x1.45mm_HandSolder, symbol Device:C_Small
- removed C97: 8.2n, Capacitor_SMD:C_0805_2012Metric_Pad1.18x1.45mm_HandSolder, symbol Device:C_Small
- removed C98: 680p, Capacitor_SMD:C_0805_2012Metric_Pad1.18x1.45mm_HandSolder, symbol Device:C_Small
- removed C99: 470p, Capacitor_SMD:C_0805_2012Metric_Pad1.18x1.45mm_HandSolder, symbol Device:C_Small
- removed L7: 4.7u, Inductor_SMD_Wurth:L_Wurth_WE-LQSH-2010, symbol Device:L
- removed Q13, Q7: CSD19502Q5B, Package_TO_SOT_SMD:TDSON-8-1, symbol Transistor_FET:CSD19502Q5B
- removed R71, R72, R73, R74, R75, R76, R77, R78, R79, R80, R81: 150K_0603, PCM_4ms_Resistor:R_0805_2012Metric, symbol PCM_4ms_Resistor:150K_0603
- removed U9: LM25145RGYR, Project_Star_Regulator_Switching:RGY0020B, symbol Project_Star_Regulator_Switching:LM25145
Connections:
- no-connect marks 1 -> 0
Other:
- note removed: "22V-33.6V to 6.00V @ 10A"
