File: hexapod_legs.kicad_sch (KiCad schematic)
At the start: 72 parts, among them J10 Leg3 Motor1, J11 Leg4 Motor3, J12 Leg4 Motor2, J13 Leg4 Motor1, J14 Leg5 Motor3, J15 Leg5 Motor2, J16 Leg5 Motor1, J17 Leg6 Motor3, J18 Leg6 Motor2, J19 Leg6 Motor1, J2 Leg1 Motor3, J3 Leg1 Motor2, J4 Leg1 Motor1, J5 Leg2 Motor3, J6 Leg2 Motor2, J7 Leg2 Motor1, J8 Leg3 Motor3, J9 Leg3 Motor2

Commit message: 20V line V2
Parts:
- renumbered J8 to J10, J9 to J11, J10 to J12, J11 to J13, J12 to J14, J13 to J15, J14 to J16, J15 to J17, J16 to J18, J17 to J19, J18 to J20, J19 to J21, J2 to J4, J3 to J5, J4 to J6, J5 to J7, J6 to J8, J7 to J9
Changed lines of the file:
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@@
 		(dnp no)
 		(fields_autoplaced yes)
-		(property "Reference" "J18"
+		(property "Reference" "J20"
 			(at 332.105 147.32 0)
 			(effects
@@
 			(project "Project-Star"
 				(path "/dfa3d008-01ec-4328-886a-a4a57a49a859/50ec6b1a-f906-43ba-9be1-78681b5bb3a1/c3b9a73c-7ccc-44f3-bc7d-7a0ac759ea5d"
-					(reference "J18")
+					(reference "J20")
 					(unit 1)
 				)
@@
 		(on_board no)
 		(dnp no)
-		(property "Reference" "J7"
+		(property "Reference" "J9"
 			(at 104.775 119.38 0)
 			(effects
@@
 			(project "Project-Star"
 				(path "/dfa3d008-01ec-4328-886a-a4a57a49a859/50ec6b1a-f906-43ba-9be1-78681b5bb3a1/c3b9a73c-7ccc-44f3-bc7d-7a0ac759ea5d"
-					(reference "J7")
+					(reference "J9")
 					(unit 1)
 				)
@@
 		(dnp no)
 		(fields_autoplaced yes)
-		(property "Reference" "J15"
+		(property "Reference" "J17"
 			(at 274.955 147.32 0)
 			(effects
@@
 			(project "Project-Star"
 				(path "/dfa3d008-01ec-4328-886a-a4a57a49a859/50ec6b1a-f906-43ba-9be1-78681b5bb3a1/c3b9a73c-7ccc-44f3-bc7d-7a0ac759ea5d"
-					(reference "J15")
+					(reference "J17")
 					(unit 1)
 				)
@@
 		(dnp no)
 		(fields_autoplaced yes)
-		(property "Reference" "J2"
+		(property "Reference" "J4"
 			(at 45.085 172.72 0)
 			(effects
@@
 			(project "Project-Star"
 				(path "/dfa3d008-01ec-4328-886a-a4a57a49a859/50ec6b1a-f906-43ba-9be1-78681b5bb3a1/c3b9a73c-7ccc-44f3-bc7d-7a0ac759ea5d"
-					(reference "J2")
+					(reference "J4")
 					(unit 1)
 				)
@@
 		(dnp no)
 		(fields_autoplaced yes)
-		(property "Reference" "J12"
+		(property "Reference" "J14"
 			(at 216.535 146.05 0)
 			(effects
@@
 			(project "Project-Star"
 				(path "/dfa3d008-01ec-4328-886a-a4a57a49a859/50ec6b1a-f906-43ba-9be1-78681b5bb3a1/c3b9a73c-7ccc-44f3-bc7d-7a0ac759ea5d"
-					(reference "J12")
+					(reference "J14")
 					(unit 1)
 				)
@@
 		(dnp no)
 		(fields_autoplaced yes)
-		(property "Reference" "J11"
+		(property "Reference" "J13"
 			(at 215.265 172.72 0)
 			(effects
@@
 			(project "Project-Star"
 				(path "/dfa3d008-01ec-4328-886a-a4a57a49a859/50ec6b1a-f906-43ba-9be1-78681b5bb3a1/c3b9a73c-7ccc-44f3-bc7d-7a0ac759ea5d"
-					(reference "J11")
+					(reference "J13")
 					(unit 1)
 				)
@@
 		(on_board no)
 		(dnp no)
-		(property "Reference" "J6"
+		(property "Reference" "J8"
 			(at 103.505 146.05 0)
 			(effects
@@
 			(project "Project-Star"
 				(path "/dfa3d008-01ec-4328-886a-a4a57a49a859/50ec6b1a-f906-43ba-9be1-78681b5bb3a1/c3b9a73c-7ccc-44f3-bc7d-7a0ac759ea5d"
-					(reference "J6")
+					(reference "J8")
 					(unit 1)
 				)
@@
 		(dnp no)
 		(fields_autoplaced yes)
-		(property "Reference" "J17"
+		(property "Reference" "J19"
 			(at 330.835 173.99 0)
 			(effects
@@
 			(project "Project-Star"
 				(path "/dfa3d008-01ec-4328-886a-a4a57a49a859/50ec6b1a-f906-43ba-9be1-78681b5bb3a1/c3b9a73c-7ccc-44f3-bc7d-7a0ac759ea5d"
-					(reference "J17")
+					(reference "J19")
 					(unit 1)
 				)
@@
 		(dnp no)
 		(fields_autoplaced yes)
-		(property "Reference" "J16"
+		(property "Reference" "J18"
 			(at 276.225 120.65 0)
 			(effects
@@
 			(project "Project-Star"
 				(path "/dfa3d008-01ec-4328-886a-a4a57a49a859/50ec6b1a-f906-43ba-9be1-78681b5bb3a1/c3b9a73c-7ccc-44f3-bc7d-7a0ac759ea5d"
-					(reference "J16")
+					(reference "J18")
 					(unit 1)
 				)
@@
 		(on_board no)
 		(dnp no)
-		(property "Reference" "J5"
+		(property "Reference" "J7"
 			(at 102.235 172.72 0)
 			(effects
@@
 			(project "Project-Star"
 				(path "/dfa3d008-01ec-4328-886a-a4a57a49a859/50ec6b1a-f906-43ba-9be1-78681b5bb3a1/c3b9a73c-7ccc-44f3-bc7d-7a0ac759ea5d"
-					(reference "J5")
+					(reference "J7")
 					(unit 1)
 				)
@@
 		(dnp no)
 		(fields_autoplaced yes)
-		(property "Reference" "J3"
+		(property "Reference" "J5"
 			(at 46.355 146.05 0)
 			(effects
@@
 			(project "Project-Star"
 				(path "/dfa3d008-01ec-4328-886a-a4a57a49a859/50ec6b1a-f906-43ba-9be1-78681b5bb3a1/c3b9a73c-7ccc-44f3-bc7d-7a0ac759ea5d"
-					(reference "J3")
+					(reference "J5")
 					(unit 1)
 				)
@@
 		(dnp no)
 		(fields_autoplaced yes)
-		(property "Reference" "J8"
+		(property "Reference" "J10"
 			(at 158.115 172.72 0)
 			(effects
@@
 			(project "Project-Star"
 				(path "/dfa3d008-01ec-4328-886a-a4a57a49a859/50ec6b1a-f906-43ba-9be1-78681b5bb3a1/c3b9a73c-7ccc-44f3-bc7d-7a0ac759ea5d"
-					(reference "J8")
+					(reference "J10")
 					(unit 1)
 				)
@@
 		(dnp no)
 		(fields_autoplaced yes)
-		(property "Reference" "J19"
+		(property "Reference" "J21"
 			(at 333.375 120.65 0)
 			(effects
@@
 			(project "Project-Star"
 				(path "/dfa3d008-01ec-4328-886a-a4a57a49a859/50ec6b1a-f906-43ba-9be1-78681b5bb3a1/c3b9a73c-7ccc-44f3-bc7d-7a0ac759ea5d"
-					(reference "J19")
+					(reference "J21")
 					(unit 1)
 				)
@@
 		(dnp no)
 		(fields_autoplaced yes)
-		(property "Reference" "J10"
+		(property "Reference" "J12"
 			(at 160.655 119.38 0)
 			(effects
@@
 			(project "Project-Star"
 				(path "/dfa3d008-01ec-4328-886a-a4a57a49a859/50ec6b1a-f906-43ba-9be1-78681b5bb3a1/c3b9a73c-7ccc-44f3-bc7d-7a0ac759ea5d"
-					(reference "J10")
+					(reference "J12")
 					(unit 1)
 				)
@@
 		(dnp no)
 		(fields_autoplaced yes)
-		(property "Reference" "J9"
+		(property "Reference" "J11"
 			(at 159.385 146.05 0)
 			(effects
@@
 			(project "Project-Star"
 				(path "/dfa3d008-01ec-4328-886a-a4a57a49a859/50ec6b1a-f906-43ba-9be1-78681b5bb3a1/c3b9a73c-7ccc-44f3-bc7d-7a0ac759ea5d"
-					(reference "J9")
+					(reference "J11")
 					(unit 1)
 				)
@@
 		(dnp no)
 		(fields_autoplaced yes)
-		(property "Reference" "J4"
+		(property "Reference" "J6"
 			(at 47.625 119.38 0)
 			(effects
@@
 			(project "Project-Star"
 				(path "/dfa3d008-01ec-4328-886a-a4a57a49a859/50ec6b1a-f906-43ba-9be1-78681b5bb3a1/c3b9a73c-7ccc-44f3-bc7d-7a0ac759ea5d"
-					(reference "J4")
+					(reference "J6")
 					(unit 1)
 				)
@@
 		(dnp no)
 		(fields_autoplaced yes)
-		(property "Reference" "J13"
+		(property "Reference" "J15"
 			(at 217.805 119.38 0)
 			(effects
@@
 			(project "Project-Star"
 				(path "/dfa3d008-01ec-4328-886a-a4a57a49a859/50ec6b1a-f906-43ba-9be1-78681b5bb3a1/c3b9a73c-7ccc-44f3-bc7d-7a0ac759ea5d"
-					(reference "J13")
+					(reference "J15")
 					(unit 1)
 				)
@@
 		(dnp no)
 		(fields_autoplaced yes)
-		(property "Reference" "J14"
+		(property "Reference" "J16"
 			(at 273.685 173.99 0)
 			(effects
@@
 			(project "Project-Star"
 				(path "/dfa3d008-01ec-4328-886a-a4a57a49a859/50ec6b1a-f906-43ba-9be1-78681b5bb3a1/c3b9a73c-7ccc-44f3-bc7d-7a0ac759ea5d"
-					(reference "J14")
+					(reference "J16")
 					(unit 1)
 				)
