File: Project-Star.kicad_sch (KiCad schematic)
At the start: 200 parts, among them J1 Conn_01x02, J2 Conn_02x04, J3 Conn_01x09, J4 Screw_Terminal_01x02, Q1 CSD13380F3, Q10 Q_NMOS, Q11 Q_NMOS, Q12 Q_PMOS, Q13 Q_PMOS, Q14 Q_NMOS, Q15 Q_NMOS, Q16 Q_NMOS, Q17 Q_NMOS, Q18 Q_NPN, Q19 Q_PMOS, Q2 CSD13380F3, Q20 TP0610K, Q21 2N7002E, Q3 CSD13380F3, Q4 CSD13380F3, Q5 CSD13380F3, Q6 CSD13380F3, Q7 CSD13380F3, Q8 CSD13380F3, Q9 2N7002E, SW1 SW_Push, U1 BQ7693000DBT, U2 TPS3839DBZ, U3 BQ76200PW, U4 LMT01LPG, U5 MSP430G2553IPW20

Commit message: redesign with refernce
Parts:
- removed C25, C26, C32: 1u, symbol Device:C
- removed C27, C28, C33, C36: 100n, symbol Device:C
- removed C29: 1.5u, symbol Device:C
- removed C30, C31: 1n, symbol Device:C
- removed C34: 2200p, symbol Device:C
- removed C37: 4u7, symbol Device:C
- removed D10, D11, D13, D9: 100V, symbol Device:D_Filled
- removed D12: 200V, symbol Device:D_Filled
- removed D14, D15, D16: 3V9, symbol Device:D_Zener_Filled
- removed D20, D21, D22, D23: GREEN, LED_THT:LED_D5.0mm, symbol PCM_SL_Devices:LED
- removed D24, D25, D26, D27, D28, D29, D3, D5, D6, D8: 5V6, symbol Device:D_Zener_Filled
- removed F2: 50V, 30A, Slow Blow, symbol PCM_Device_AKL:Fuse
- removed FB1, FB2, FB3, FB4: 200R, symbol Device:FerriteBead
- removed J2: Conn_02x04, 4ms_Connector:Pins_2x04_2.54mm_TH, symbol PCM_4ms_Connector:Conn_02x04
- removed J3: Conn_01x09, 4ms_Connector:Pins_1x09_2.54mm_TH, symbol PCM_4ms_Connector:Conn_01x09
- removed J4: Screw_Terminal_01x02, symbol Connector:Screw_Terminal_01x02
- removed NT1, NT2, NT3: NetTie, symbol Device:NetTie_2
- removed NTC1, NTC2: 10k, symbol Device:Thermistor
- removed Q1, Q2, Q3, Q4, Q5, Q6, Q7, Q8: CSD13380F3, Package_DFN_QFN:Texas_PicoStar_DFN-3_0.69x0.60mm, symbol Transistor_FET:CSD13380F3
- removed Q10, Q11, Q14, Q15, Q16, Q17: Q_NMOS, symbol Device:Q_NMOS
- removed Q12, Q13, Q19: Q_PMOS, symbol Device:Q_PMOS
- removed Q18: Q_NPN, symbol Device:Q_NPN
- removed Q20: TP0610K, PCM_Package_TO_SOT_SMD_AKL:SOT-23, symbol PCM_Transistor_MOSFET_AKL:TP0610K
- removed Q21, Q9: 2N7002E, PCM_Package_TO_SOT_SMD_AKL:SOT-23, symbol PCM_Transistor_MOSFET_AKL:2N7002E
- removed R51: 1k2, symbol Device:R
- removed R52, R53, R54: 10M, symbol Device:R
- removed R55, R56, R57: 620R, symbol Device:R
- removed R58, R59, R61, R75, R76, R77, R78, R79, R80, R81, R82, R83, R84, R85, R86: 100R, symbol Device:R
- removed R60, R63: 0R, symbol Device:R
- removed R62: 750, symbol Device:R
- removed R64, R67, R68, R69, R70, R71: 1k, symbol Device:R
- removed R65, R73, R74, R90: 10k, symbol Device:R
- removed R66: 154k, symbol Device:R
- removed R72: 3k, symbol Device:R
- removed R87, R88, R91: 100k, symbol Device:R
- removed R89: 130k, symbol Device:R
- removed SW1: SW_Push, symbol Switch:SW_Push
- removed TVS1: SMAJ40A, Diode_SMD:D_SMA, symbol Diode:SMAJ40A
- removed TVS2, TVS3: 5.0SMDJ36A, Diode_SMD:D_SMC, symbol Diode:Z3SMCxxx
- removed U2: TPS3839DBZ, Package_TO_SOT_SMD:SOT-23, symbol Power_Supervisor:TPS3839DBZ
- removed U3: BQ76200PW, Package_SO:TSSOP-16_4.4x5mm_P0.65mm, symbol Battery_Management:BQ76200PW
- removed U4: LMT01LPG, Package_TO_SOT_THT:TO-92-2, symbol Sensor_Temperature:LMT01LPG
- removed U5: MSP430G2553IPW20, Package_SO:TSSOP-20_4.4x6.5mm_P0.65mm, symbol MCU_Texas_MSP430:MSP430G2553IPW20
- added D10, D12, D14, D15, D3, D5, D6, D8: LED, LED_THT:LED_D5.0mm, symbol PCM_SL_Devices:LED
- added D11: 3V3, symbol Device:D_Zener_Filled
- added D13, D20, D9: 5V6, symbol Device:D_Zener_Filled
- added D16: 1N4148W, PCM_Diode_SMD_AKL:D_SOD-123, symbol PCM_Diode_AKL:1N4148W
- added J2: J_TH2, 4ms_Connector:Pins_1x02_2.54mm_TH, symbol PCM_4ms_Connector:Conn_01x02
- added J3: J_BOOT, 4ms_Connector:Pins_1x02_2.54mm_TH, symbol PCM_4ms_Connector:Conn_01x02
- added Q1, Q2, Q3, Q4, Q6, Q7, Q8, Q9: DMN2004K, PCM_Package_TO_SOT_SMD_AKL:SOT-23, symbol PCM_Transistor_MOSFET_AKL:DMN2004K
- added Q5: CSD19531Q5A, Package_TO_SOT_SMD:TDSON-8-1, symbol Transistor_FET:CSD19531Q5A
- added SW1: BOOT, Button_Switch_THT:SW_PUSH_6mm, symbol PCM_SL_Devices:Push_Button
- added TH1, TH2: 10k NTC, symbol Device:Thermistor
- added U2: BQ76200PW, Package_SO:TSSOP-16_4.4x5mm_P0.65mm, symbol Battery_Management:BQ76200PW
- C1, C10, C2, C3, C4, C5, C6, C8, C9: value 220n -> 100n
- C11, C21: value 4700p -> 100n
- C12: value 1u -> 10u
- C13: value 100n -> 1u
- C14: value 100n -> 4u7
- C15: value 4u7 -> 4n7
- C17: value 10u -> 4n7
- C18: value 10u -> 1u
- C19, C20: value 1u -> 100n
- C22: value 1u -> 10n
- C23: value 470p -> 10n
- C7: value 220n -> 1u
- D17: value 16V -> 3V3
- D18: value 16V -> 5V6
- D19: value 18V -> 5V6
- D2: value 5V6 -> 3V3
- J1: value Conn_01x02 -> J_TH1
- R12, R21, R22, R4: value 28R7 -> 1k
- R13: value 1k -> 33R
- R15, R38, R5: value 1k -> 10k
- R16, R29, R6: value 10k -> 1k
- R17, R3, R9: value 28R7 -> 33R
- R19: value 10k -> 100R
- R20: value 28R7 -> 510k
- R26, R30, R8: value 10k -> 33R
- R28: value 3M -> 33R
- R31: value 510k -> 1k
- R32: value 100k -> 1k
- R33: value 100R -> 4k7
- R34: value 100k -> 4k7
- R35: value 1k -> 4k7
- R36: value 3M -> 100R
- R39: value 51k -> 1k
- R40: value 10M -> 10k
- R41: value 1M -> 1k
- R42: value 100k -> 10k
- R43: value 10M -> 100R
- R44, R45: value 0R -> 1k
- R46: value 100R -> 1k
- R48: value 1k2 -> 100R
- R49, R50: value 1k2 -> 4R7
Connections:
- net CGATE is gone; now on net SRN: D17.1 (K)
- net DGATE is gone; now on an unnamed net: D18.1 (K)
- net SNSN is gone; now on net U_BAT: R47.1
- net SNSP is gone; now on net CHG_EN: R46.1
- net WAKE is gone; now on net VC7: R38.2
- net +BATT: now also R47.2; no longer C23.2, R20.2, R23.1, R34.2, R35.1
- net ALERT: now also R32.2; no longer C16.1, R31.1, U1.30 (ALERT)
- net BAT: now also C7.2, R19.2, U1.15 (BAT)
- net C1: now also D4.2 (A), R35.1, R6.1, D3.2, Q2.2 (S); no longer D2.2 (A), R5.1
- net C2: now also D7.2 (A), R12.1, R8.1, D5.2, Q3.2 (S); no longer R4.2, R7.1
- net C3: now also R22.1, R9.1, D6.2, D9.2 (A), Q4.2 (S); no longer D4.2 (A), R10.1, R9.2
- net C4: now also R16.1, R23.1, D8.2; no longer R12.2, R14.1, R15.1
- net C5: now also R17.1, R21.1, D10.2, D16.2 (A), D20.2 (A), Q9.2 (S); no longer R17.2, R18.1
- net C6: now also D19.2 (A), R30.1, R41.1, D15.2, Q8.2 (S); no longer R22.2, R27.1
- net C7: now also D18.2 (A), R28.1, R39.1, D14.2, Q7.2 (S); no longer D7.2 (A), R21.2, R25.1
- net CHG: now also U1.2 (CHG)
- net CHG_EN: no longer U1.2 (CHG)
- net DSG: now also U1.1 (DSG); no longer D19.1 (K)
- net DSG_EN: now also R45.1; no longer U1.1 (DSG)
- net GND: now also C1.1, C12.1, C13.1, C14.1, C19.2, C2.2, C21.1, C23.2, C7.1, D17.2 (A), D2.2 (A), J1.2 (Pin_2), R20.2, D11.2 (A), TH1.2, U2.5 (CP_EN), U2.7 (PMON_EN), U2.9 (VSS); no longer C1.2, C17.1, C19.1, C20.1, C21.2, C24.2, R31.2, R36.2, R40.1
- net PCHG_EN: now also R44.1
- net REGOUT: now also C14.2; no longer C15.1, R29.2, R30.2, R42.2
- net REGSRC: now also C12.2; no longer C19.2
- net SCL: now also R34.1; no longer R30.1
- net SDA: now also R33.1; no longer R29.1
- net TS1: now also C15.1, J1.1 (Pin_1), J3.2 (Pin_2), SW1.2, TH1.1; no longer C21.1, R36.1
- net VCX5: now also C8.2, R16.2, J2.2 (Pin_2), TH2.2; no longer C11.2, C12.2, C18.1, C7.2, R14.2, R28.2, R32.2, R35.2, U1.15 (BAT)
- net C8: now reaches R37.1
- net C8: now also R26.1, D12.2; no longer R39.1
- net at R32.1: now also C16.1, R20.1, U1.30 (ALERT)
- net VC0: now reaches D2.1 (K)
- net VC0: now also C1.2, R1.2, R2.2, U1.27 (VC0); no longer R6.1
- net VC1: now reaches C2.1, C3.2, R5.2, R6.2, U1.26 (VC1)
- net VC6: now reaches R40.2
- net VC6: now also C10.2, C11.1, R41.2, U1.19 (VC7); no longer R41.1
- net at D7.1 (K): now also R11.1, Q3.1 (G); no longer R24.1
- net at D1.1 (K), R1.1: now also Q1.1 (G)
- net at D4.1 (K): now also R5.1, Q2.1 (G); no longer R11.1
- net at R4.1: now also D3.1
- net SRN: now reaches C20.2
- net SRN: now also C19.1, R43.2, U1.29 (SRN); no longer R33.1
- net VC3: now reaches C4.1, C5.2, U1.23 (VC4), U1.24 (VC3)
- net VC3: now also R15.2, R22.2; no longer R10.2, R11.2
- net at C23.1: now also R48.2, U2.11 (PACK); no longer R43.1
- net at R42.1: now also D20.1 (K), Q9.1 (G)
- net at R19.1: now also D16.1 (K)
- net VC4: now reaches C5.1, U1.22 (VC5)
- net VC4: now also R23.2; no longer R13.2
- net CAP2: now reaches U1.11 (NC(CAP2)), U1.12 (NC(CAP2)), U1.14 (CAP2)
- net CAP2: no longer C12.1
- net VC2: now reaches C3.1, C4.2, U1.25 (VC2)
- net VC2: now also R11.2, R12.2; no longer R7.2, R8.2
- net VC5B: now reaches C6.1, U1.21 (VC5B)
- net VC5B: now also R24.2, R25.2; no longer R15.2, R16.2
- net at R38.1: now also Q7.1 (G); no longer R37.2
- net CAP1: now reaches C13.2
- net CAP1: now also U1.7 (CAP1); no longer C14.1
- net VC7: now reaches R39.2
- net VC7: now also C10.1, C9.2, U1.17 (VC9), U1.18 (VC8)
- net U_BAT: now reaches C22.1
- net U_BAT: now also C24.2, U2.2 (BAT); no longer U1.7 (CAP1)
- net at R3.1: now also R4.2, Q1.3 (D)
- net +3.3V: now reaches R33.2
- net +3.3V: now also R34.2; no longer R34.1
- net -BATT renamed C0
- net C0: now also Q1.2 (S); no longer R44.1, R45.1
- removed net ISENSE: R47.2, U1.29 (SRN)
- removed net PACK+: C13.1, D18.2 (A), R43.2
- removed net PACK-: C14.2, R44.2, R45.2
- removed net PDRAIN: R48.2, R49.2, R50.2
- new net: D15.1, R31.1
- new net: Q9.3 (D), R30.2, R31.2
- new net: Q6.3 (D), R17.2, R18.2
- new net: D19.1 (K), Q8.1 (G), R40.1
- new net: Q8.3 (D), R28.2, R29.2
- new net: R50.1, U2.16 (CHG)
- new net: D13.1 (K), Q6.1 (G), R24.1
- new net: D13.2 (A), Q6.2 (S), R25.1
- new net: Q2.3 (D), R7.2, R8.2
- new net: D14.1, R29.1
- new net: R46.2, U2.4 (CHG_EN)
- new net: D12.1, R27.1
- new net: Q7.3 (D), R26.2, R27.2
- new net: D5.1, R7.1
- new net: D8.1, R14.1
- new net: Q4.3 (D), R13.2, R14.2
- new net: C24.1, U2.1 (VDDCP)
- new net: R49.1, U2.12 (DSG)
- new net: R45.2, U2.6 (DSG_EN)
- new net: R44.2, U2.8 (PCHG_EN)
- new net: Q3.3 (D), R10.2, R9.2
- new net: D9.1 (K), Q4.1 (G), R15.1
- new net: J3.1 (Pin_1), R35.2, SW1.1
- new net: Q5.1 (S), Q5.2 (S), Q5.3 (S)
- new net: D6.1, R10.1
- new net: D10.1, R18.1
- new net +PACK: R48.1
- new net G_CHG: R50.2
- new net G_DSG: R49.2
- new net G_PCHG: U2.14 (PCHG)
- new net R_SENSE+: R36.1
- new net R_SENSE-: R43.1
- new net SRP: C20.1, C21.2, D11.1 (K), R36.2, U1.28 (SRP)
- new net TS2: C17.1, C18.1, J2.1 (Pin_1), TH2.1, U1.13 (TS2)
- new net VC5: C11.2, C8.1, R21.2, R42.2, U1.20 (VC6)
- new net VC8: C9.1, R37.2, U1.16 (VC10)
- no-connect marks 0 -> 1
Other:
- added sheet bk (bk.kicad_sch)
- note added: ">1 for boot-up"
- note added: "Balancing & BMC"
- note added: "Boot Switch"
- note added: "Current Sense Filtering"
- note added: "From slva729a VDDCP was picked"
- note added: "High-Side Gate Driver"
- note added: "I2C Pullups"
- note added: "Interrupt for new current readings or errors"
- note added: "Passive Balancing Circuit"
- note added: "REGOUT +3V3 Iout max 40mA"
- note added: "TODO: Look at the doc for more boot switch options"
- note added: "Thermistors"
- note added: "VC0-VSS (Vin max 3V6)"

Commit message: datasheets
Parts:
- removed J3: J_BOOT, 4ms_Connector:Pins_1x02_2.54mm_TH, symbol PCM_4ms_Connector:Conn_01x02
- removed SW1: BOOT, Button_Switch_THT:SW_PUSH_6mm, symbol PCM_SL_Devices:Push_Button
- added C25, C29, C30: 4u7, symbol Device:C
- added C26: 2n2, symbol Device:C
- added C27: 3n3, symbol Device:C
- added C28: 56p, symbol Device:C
- added C31: 100n, symbol Device:C
- added C32: 2u2, symbol Device:C
- added D21, D22: MBR0520LT1G, symbol PCM_Diode_Schottky_AKL:D_Schottky_Generic
- added D23: 16V, symbol Device:D_Zener_Filled
- added D24: 18V, symbol Device:D_Zener_Filled
- added D25, D26, D28: 1N4148W, PCM_Diode_SMD_AKL:D_SOD-123, symbol PCM_Diode_AKL:1N4148W
- added D27: 3V3, symbol Device:D_Zener_Filled
- added D29: GREEN, LED_THT:LED_D5.0mm, symbol PCM_SL_Devices:LED
- added L1: 68u, symbol Device:L
- added Q10: CSD18540Q5B, Package_TO_SOT_SMD:TDSON-8-1, symbol Transistor_FET:CSD18540Q5B
- added Q11, Q13: ZXMP10A13F, PCM_Package_TO_SOT_SMD_AKL:SOT-23, symbol PCM_Transistor_MOSFET_AKL:ZXMP10A13F
- added Q12: BSS123, PCM_Package_TO_SOT_SMD_AKL:SOT-23, symbol PCM_Transistor_MOSFET_AKL:BSS123
- added R51, R65: 1k, symbol Device:R
- added R52: 715k, symbol Device:R
- added R53, R59: 1M, symbol Device:R
- added R54: 115k, symbol Device:R
- added R55, R60: 10M, symbol Device:R
- added R56: 3M, symbol Device:R
- added R57: 383k, symbol Device:R
- added R58: 240k, symbol Device:R
- added R61: 360k, symbol Device:R
- added R62: 10k, symbol Device:R
- added R63: 100, symbol Device:R
- added R64: 3k01, symbol Device:R
- added SW1: SW_SPST, symbol Switch:SW_SPST
- added U3: LM5164DDA, Package_SO:HSOP-8-1EP_3.9x4.9mm_P1.27mm_EP2.41x3.1mm_ThermalVias, symbol Regulator_Switching:LM5164DDA
- R19: value 100R -> 1k
- R35: value 4k7 -> 6M8
- U1: value BQ7693000DBT -> BQ7693006DBTR
Connections:
- net REGOUT is gone; now on net +3V3: C14.2, U1.8 (REGOUT)
- net BAT: now also D16.1 (K)
- net C1: now also R64.2; no longer R35.1
- net C5: no longer D16.2 (A)
- net C8: now also R19.1, C31.2, D23.1 (K), Q11.2 (S), R56.2
- net CHG_EN: now also R51.1
- net GND: now also C25.2, C29.1, C30.1, D29.1, Q12.2 (S), R53.1, R54.1, R55.1, R58.1, U3.1 (GND), U3.9 (EP); no longer U2.5 (CP_EN)
- net TS1: now also D26.1 (K), SW1.2 (B)
- net VC4: now also D25.2 (A)
- net VC8: now also D16.2 (A)
- net VCX5: no longer C6.2, C8.2, R16.2, U1.10 (VC5X)
- net at R35.2: now also D23.2 (A), Q11.1 (G), R56.1
- net +3.3V renamed +3V3
- net +3V3: now also D22.2 (A), R65.1
- net +PACK renamed PACK+
- net PACK+: now also D24.1 (K), Q13.2 (S), R59.2
- new net: D21.1 (K), D22.1 (K), Q12.1 (G), R55.2
- new net: C25.1, Q11.3 (D), U3.2 (VIN), U3.3 (EN/UVLO)
- new net: R53.2, R54.2, U3.4 (RON)
- new net: C28.2, U3.5 (FB)
- new net: C26.1, L1.1, U3.7 (BST)
- new net: C26.2, R57.1, U3.8 (SW)
- new net: Q10.1 (S), Q10.2 (S), Q10.3 (S)
- new net: Q12.3 (D), R35.1
- new net: D26.2 (A), D27.1 (K), D28.1 (K), R61.1, R62.2
- new net: D29.2, R65.2
- new net: R64.1, SW1.1 (A)
- new net: R51.2, U2.5 (CP_EN)
- new net: C27.1, C28.1, R52.1, R57.2, R58.2
- new net: C31.1, D24.2 (A), Q13.1 (G), R59.1
- new net: C32.1, R60.2, R61.2
- new net: C32.2, Q13.3 (D), R60.1
- new net: D28.2 (A), R63.2
- new net 430_PWR: D21.2 (A)
- new net 5V: C27.2, C29.2, C30.2, L1.2, R52.2
- new net PACK-: D27.2 (A), R62.1
- new net VC5X: C6.2, C8.2, D25.1 (K), R16.2, U1.10 (VC5X)
- new net WAKE: R63.1
- no-connect marks 1 -> 2
Other:
- note added: "5V Supply"
- note added: "REGOUT supplys 3v3"
- note added: "Wake-Up"
- note added: "from TIDA-010030"
- note added: "system is on LED"
- note removed: ">1 for boot-up"
- note removed: "Boot Switch"
- note removed: "REGOUT +3V3 Iout max 40mA"
- note removed: "TODO: Look at the doc for more boot switch options"
- moved on the sheet: C22, D16
