File: BMS Read Voltage.kicad_sch (KiCad schematic)
At the start: 8 parts, among them Q34 BSS138, Q36 TP0610K-T1-GE3

Commit message: worked on MCU
Parts:
- renumbered D58 to D30, Q34 to Q17, Q36 to Q18, R168 to R75, R173 to R76, R174 to R77, R177 to R78, R178 to R79
Connections:
- net PACK_READ_TMP renamed PACK_READ_STATS
Other:
- note added: "TODO: Find out what this is for"
Changed lines of the file:
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@@
 	(generator_version "9.0")
 	(paper "A4")
+	(text "TODO: Find out what this is for"
+		(exclude_from_sim no)
+		(at 141.478 116.586 0)
+		(effects
+			(font
+				(size 1.27 1.27)
+			)
+		)
+	)
 	(text "Read \nVoltage"
 		(exclude_from_sim no)
@@
 		)
 	)
-	(label "PACK_READ_TMP"
-		(at 113.03 97.79 0)
+	(label "PACK_READ_STATS"
+		(at 111.76 97.79 0)
 		(effects
 			(font
@@
 		)
 	)
-	(hierarchical_label "PACK_READ_TMP"
+	(hierarchical_label "PACK_READ_STATS"
 		(shape input)
 		(at 107.95 97.79 180)
@@
 		(on_board yes)
 		(dnp no)
-		(property "Reference" "R177"
+		(property "Reference" "R78"
 			(at 145.542 85.344 0)
 			(effects
@@
 			(project "Project-Star"
 				(path "/fc8533bc-25dd-4c20-9b4c-ffebebd6739b/e8da5d81-614b-4fe5-84b3-4c351fab7114/bad915fd-f1b0-44f5-8fcf-8d1c33cbafd0"
-					(reference "R177")
+					(reference "R78")
 					(unit 1)
 				)
@@
 		(on_board yes)
 		(dnp no)
-		(property "Reference" "R178"
+		(property "Reference" "R79"
 			(at 145.542 95.504 0)
 			(effects
@@
 			(project "Project-Star"
 				(path "/fc8533bc-25dd-4c20-9b4c-ffebebd6739b/e8da5d81-614b-4fe5-84b3-4c351fab7114/bad915fd-f1b0-44f5-8fcf-8d1c33cbafd0"
-					(reference "R178")
+					(reference "R79")
 					(unit 1)
 				)
@@
 		(on_board yes)
 		(dnp no)
-		(property "Reference" "#PWR064"
+		(property "Reference" "#PWR019"
 			(at 113.03 115.57 0)
 			(effects
@@
 			(project "Project-Star"
 				(path "/fc8533bc-25dd-4c20-9b4c-ffebebd6739b/e8da5d81-614b-4fe5-84b3-4c351fab7114/bad915fd-f1b0-44f5-8fcf-8d1c33cbafd0"
-					(reference "#PWR064")
+					(reference "#PWR019")
 					(unit 1)
 				)
@@
 		(on_board yes)
 		(dnp no)
-		(property "Reference" "Q36"
+		(property "Reference" "Q18"
 			(at 143.764 75.184 0)
 			(effects
@@
 			(project "Project-Star"
 				(path "/fc8533bc-25dd-4c20-9b4c-ffebebd6739b/e8da5d81-614b-4fe5-84b3-4c351fab7114/bad915fd-f1b0-44f5-8fcf-8d1c33cbafd0"
-					(reference "Q36")
+					(reference "Q18")
 					(unit 1)
 				)
@@
 		(on_board yes)
 		(dnp no)
-		(property "Reference" "R173"
+		(property "Reference" "R76"
 			(at 135.382 70.104 0)
 			(effects
@@
 			(project "Project-Star"
 				(path "/fc8533bc-25dd-4c20-9b4c-ffebebd6739b/e8da5d81-614b-4fe5-84b3-4c351fab7114/bad915fd-f1b0-44f5-8fcf-8d1c33cbafd0"
-					(reference "R173")
+					(reference "R76")
 					(unit 1)
 				)
@@
 		(on_board yes)
 		(dnp no)
-		(property "Reference" "Q34"
+		(property "Reference" "Q17"
 			(at 133.604 92.456 0)
 			(effects
@@
 			(project "Project-Star"
 				(path "/fc8533bc-25dd-4c20-9b4c-ffebebd6739b/e8da5d81-614b-4fe5-84b3-4c351fab7114/bad915fd-f1b0-44f5-8fcf-8d1c33cbafd0"
-					(reference "Q34")
+					(reference "Q17")
 					(unit 1)
 				)
@@
 		(on_board yes)
 		(dnp no)
-		(property "Reference" "R174"
+		(property "Reference" "R77"
 			(at 135.382 82.804 0)
 			(effects
@@
 			(project "Project-Star"
 				(path "/fc8533bc-25dd-4c20-9b4c-ffebebd6739b/e8da5d81-614b-4fe5-84b3-4c351fab7114/bad915fd-f1b0-44f5-8fcf-8d1c33cbafd0"
-					(reference "R174")
+					(reference "R77")
 					(unit 1)
 				)
@@
 		(on_board yes)
 		(dnp no)
-		(property "Reference" "D58"
+		(property "Reference" "D30"
 			(at 153.67 96.774 90)
 			(effects
@@
 			(project "Project-Star"
 				(path "/fc8533bc-25dd-4c20-9b4c-ffebebd6739b/e8da5d81-614b-4fe5-84b3-4c351fab7114/bad915fd-f1b0-44f5-8fcf-8d1c33cbafd0"
-					(reference "D58")
+					(reference "D30")
 					(unit 1)
 				)
@@
 		(on_board yes)
 		(dnp no)
-		(property "Reference" "R168"
+		(property "Reference" "R75"
 			(at 115.062 99.314 0)
 			(effects
@@
 			(project "Project-Star"
 				(path "/fc8533bc-25dd-4c20-9b4c-ffebebd6739b/e8da5d81-614b-4fe5-84b3-4c351fab7114/bad915fd-f1b0-44f5-8fcf-8d1c33cbafd0"
-					(reference "R168")
+					(reference "R75")
 					(unit 1)
 				)
@@
 		(on_board yes)
 		(dnp no)
-		(property "Reference" "#PWR085"
+		(property "Reference" "#PWR020"
 			(at 143.51 111.76 0)
 			(effects
@@
 			(project "Project-Star"
 				(path "/fc8533bc-25dd-4c20-9b4c-ffebebd6739b/e8da5d81-614b-4fe5-84b3-4c351fab7114/bad915fd-f1b0-44f5-8fcf-8d1c33cbafd0"
-					(reference "#PWR085")
+					(reference "#PWR020")
 					(unit 1)
 				)
