File: Current Sense Filtering.kicad_sch (KiCad schematic)
At the start: 7 parts

Commit message: worked on MCU
Parts:
- renumbered C57 to C16, C58 to C17, C61 to C18, D51 to D21, D54 to D22, R151 to R42, R155 to R43
Changed lines of the file:
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@@
 		(on_board yes)
 		(dnp no)
-		(property "Reference" "C61"
+		(property "Reference" "C18"
 			(at 160.02 94.234 90)
 			(effects
@@
 			(project "Project-Star"
 				(path "/fc8533bc-25dd-4c20-9b4c-ffebebd6739b/e8da5d81-614b-4fe5-84b3-4c351fab7114/ec6b8b52-e72f-4bdb-9407-1b78ccd1535b"
-					(reference "C61")
+					(reference "C18")
 					(unit 1)
 				)
@@
 		(on_board yes)
 		(dnp no)
-		(property "Reference" "D51"
+		(property "Reference" "D21"
 			(at 134.366 86.36 0)
 			(effects
@@
 			(project "Project-Star"
 				(path "/fc8533bc-25dd-4c20-9b4c-ffebebd6739b/e8da5d81-614b-4fe5-84b3-4c351fab7114/ec6b8b52-e72f-4bdb-9407-1b78ccd1535b"
-					(reference "D51")
+					(reference "D21")
 					(unit 1)
 				)
@@
 		(on_board yes)
 		(dnp no)
-		(property "Reference" "R151"
+		(property "Reference" "R42"
 			(at 144.526 98.044 0)
 			(effects
@@
 			(project "Project-Star"
 				(path "/fc8533bc-25dd-4c20-9b4c-ffebebd6739b/e8da5d81-614b-4fe5-84b3-4c351fab7114/ec6b8b52-e72f-4bdb-9407-1b78ccd1535b"
-					(reference "R151")
+					(reference "R42")
 					(unit 1)
 				)
@@
 		(on_board yes)
 		(dnp no)
-		(property "Reference" "D54"
+		(property "Reference" "D22"
 			(at 155.956 86.614 0)
 			(effects
@@
 			(project "Project-Star"
 				(path "/fc8533bc-25dd-4c20-9b4c-ffebebd6739b/e8da5d81-614b-4fe5-84b3-4c351fab7114/ec6b8b52-e72f-4bdb-9407-1b78ccd1535b"
-					(reference "D54")
+					(reference "D22")
 					(unit 1)
 				)
@@
 		(on_board yes)
 		(dnp no)
-		(property "Reference" "C58"
+		(property "Reference" "C17"
 			(at 147.32 94.234 90)
 			(effects
@@
 			(project "Project-Star"
 				(path "/fc8533bc-25dd-4c20-9b4c-ffebebd6739b/e8da5d81-614b-4fe5-84b3-4c351fab7114/ec6b8b52-e72f-4bdb-9407-1b78ccd1535b"
-					(reference "C58")
+					(reference "C17")
 					(unit 1)
 				)
@@
 		(on_board yes)
 		(dnp no)
-		(property "Reference" "#PWR063"
+		(property "Reference" "#PWR06"
 			(at 167.64 102.87 0)
 			(effects
@@
 			(project "Project-Star"
 				(path "/fc8533bc-25dd-4c20-9b4c-ffebebd6739b/e8da5d81-614b-4fe5-84b3-4c351fab7114/ec6b8b52-e72f-4bdb-9407-1b78ccd1535b"
-					(reference "#PWR063")
+					(reference "#PWR06")
 					(unit 1)
 				)
@@
 		(on_board yes)
 		(dnp no)
-		(property "Reference" "R155"
+		(property "Reference" "R43"
 			(at 157.226 98.044 0)
 			(effects
@@
 			(project "Project-Star"
 				(path "/fc8533bc-25dd-4c20-9b4c-ffebebd6739b/e8da5d81-614b-4fe5-84b3-4c351fab7114/ec6b8b52-e72f-4bdb-9407-1b78ccd1535b"
-					(reference "R155")
+					(reference "R43")
 					(unit 1)
 				)
@@
 		(on_board yes)
 		(dnp no)
-		(property "Reference" "C57"
+		(property "Reference" "C16"
 			(at 134.62 94.234 90)
 			(effects
@@
 			(project "Project-Star"
 				(path "/fc8533bc-25dd-4c20-9b4c-ffebebd6739b/e8da5d81-614b-4fe5-84b3-4c351fab7114/ec6b8b52-e72f-4bdb-9407-1b78ccd1535b"
-					(reference "C57")
+					(reference "C16")
 					(unit 1)
 				)
@@
 		(on_board yes)
 		(dnp no)
-		(property "Reference" "#PWR060"
+		(property "Reference" "#PWR05"
 			(at 129.54 102.87 0)
 			(effects
@@
 			(project "Project-Star"
 				(path "/fc8533bc-25dd-4c20-9b4c-ffebebd6739b/e8da5d81-614b-4fe5-84b3-4c351fab7114/ec6b8b52-e72f-4bdb-9407-1b78ccd1535b"
-					(reference "#PWR060")
-					(unit 1)
-				)
+					(reference "#PWR05")
+					(unit 1)
+				)
