File: High Voltage REGSRC Supply.kicad_sch (KiCad schematic)
At the start: 10 parts, among them Q35 BSS123

Commit message: worked on MCU
Parts:
- renumbered C65 to C31, C66 to C32, C67 to C33, C68 to C34, D57 to D29, Q35 to Q16, R171 to R71, R172 to R72, R175 to R73, R176 to R74
Changed lines of the file:
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@@
 	)
 	(hierarchical_label "REGSRC"
-		(shape input)
+		(shape output)
 		(at 137.16 110.49 180)
 		(effects
@@
 		(on_board yes)
 		(dnp no)
-		(property "Reference" "Q35"
+		(property "Reference" "Q16"
 			(at 152.4 100.838 0)
 			(effects
@@
 			(project "Project-Star"
 				(path "/fc8533bc-25dd-4c20-9b4c-ffebebd6739b/e8da5d81-614b-4fe5-84b3-4c351fab7114/e3d465d4-4bae-42f2-91c8-f61f15aa6ae9"
-					(reference "Q35")
+					(reference "Q16")
 					(unit 1)
 				)
@@
 		(on_board yes)
 		(dnp no)
-		(property "Reference" "#PWR065"
+		(property "Reference" "#PWR017"
 			(at 129.54 104.14 0)
 			(effects
@@
 			(project "Project-Star"
 				(path "/fc8533bc-25dd-4c20-9b4c-ffebebd6739b/e8da5d81-614b-4fe5-84b3-4c351fab7114/e3d465d4-4bae-42f2-91c8-f61f15aa6ae9"
-					(reference "#PWR065")
+					(reference "#PWR017")
 					(unit 1)
 				)
@@
 		(on_board yes)
 		(dnp no)
-		(property "Reference" "#PWR068"
+		(property "Reference" "#PWR018"
 			(at 152.4 125.73 0)
 			(effects
@@
 			(project "Project-Star"
 				(path "/fc8533bc-25dd-4c20-9b4c-ffebebd6739b/e8da5d81-614b-4fe5-84b3-4c351fab7114/e3d465d4-4bae-42f2-91c8-f61f15aa6ae9"
-					(reference "#PWR068")
+					(reference "#PWR018")
 					(unit 1)
 				)
@@
 		(on_board yes)
 		(dnp no)
-		(property "Reference" "C66"
+		(property "Reference" "C32"
 			(at 129.54 90.932 0)
 			(effects
@@
 			(project "Project-Star"
 				(path "/fc8533bc-25dd-4c20-9b4c-ffebebd6739b/e8da5d81-614b-4fe5-84b3-4c351fab7114/e3d465d4-4bae-42f2-91c8-f61f15aa6ae9"
-					(reference "C66")
+					(reference "C32")
 					(unit 1)
 				)
@@
 		(on_board yes)
 		(dnp no)
-		(property "Reference" "R175"
+		(property "Reference" "R73"
 			(at 148.082 81.534 0)
 			(effects
@@
 			(project "Project-Star"
 				(path "/fc8533bc-25dd-4c20-9b4c-ffebebd6739b/e8da5d81-614b-4fe5-84b3-4c351fab7114/e3d465d4-4bae-42f2-91c8-f61f15aa6ae9"
-					(reference "R175")
+					(reference "R73")
 					(unit 1)
 				)
@@
 		(on_board yes)
 		(dnp no)
-		(property "Reference" "R172"
+		(property "Reference" "R72"
 			(at 144.272 95.504 0)
 			(effects
@@
 			(project "Project-Star"
 				(path "/fc8533bc-25dd-4c20-9b4c-ffebebd6739b/e8da5d81-614b-4fe5-84b3-4c351fab7114/e3d465d4-4bae-42f2-91c8-f61f15aa6ae9"
-					(reference "R172")
+					(reference "R72")
 					(unit 1)
 				)
@@
 		(on_board yes)
 		(dnp no)
-		(property "Reference" "C65"
+		(property "Reference" "C31"
 			(at 129.54 82.042 0)
 			(effects
@@
 			(project "Project-Star"
 				(path "/fc8533bc-25dd-4c20-9b4c-ffebebd6739b/e8da5d81-614b-4fe5-84b3-4c351fab7114/e3d465d4-4bae-42f2-91c8-f61f15aa6ae9"
-					(reference "C65")
+					(reference "C31")
 					(unit 1)
 				)
@@
 		(on_board yes)
 		(dnp no)
-		(property "Reference" "D57"
+		(property "Reference" "D29"
 			(at 154.432 82.804 90)
 			(effects
@@
 			(project "Project-Star"
 				(path "/fc8533bc-25dd-4c20-9b4c-ffebebd6739b/e8da5d81-614b-4fe5-84b3-4c351fab7114/e3d465d4-4bae-42f2-91c8-f61f15aa6ae9"
-					(reference "D57")
+					(reference "D29")
 					(unit 1)
 				)
@@
 		(on_board yes)
 		(dnp no)
-		(property "Reference" "C67"
+		(property "Reference" "C33"
 			(at 152.4 112.522 0)
 			(effects
@@
 			(project "Project-Star"
 				(path "/fc8533bc-25dd-4c20-9b4c-ffebebd6739b/e8da5d81-614b-4fe5-84b3-4c351fab7114/e3d465d4-4bae-42f2-91c8-f61f15aa6ae9"
-					(reference "C67")
+					(reference "C33")
 					(unit 1)
 				)
@@
 		(on_board yes)
 		(dnp no)
-		(property "Reference" "C68"
+		(property "Reference" "C34"
 			(at 161.29 102.362 0)
 			(effects
@@
 			(project "Project-Star"
 				(path "/fc8533bc-25dd-4c20-9b4c-ffebebd6739b/e8da5d81-614b-4fe5-84b3-4c351fab7114/e3d465d4-4bae-42f2-91c8-f61f15aa6ae9"
-					(reference "C68")
+					(reference "C34")
 					(unit 1)
 				)
@@
 		(on_board yes)
 		(dnp no)
-		(property "Reference" "R176"
+		(property "Reference" "R74"
 			(at 154.432 90.424 0)
 			(effects
@@
 			(project "Project-Star"
 				(path "/fc8533bc-25dd-4c20-9b4c-ffebebd6739b/e8da5d81-614b-4fe5-84b3-4c351fab7114/e3d465d4-4bae-42f2-91c8-f61f15aa6ae9"
-					(reference "R176")
+					(reference "R74")
 					(unit 1)
 				)
@@
 		(on_board yes)
 		(dnp no)
-		(property "Reference" "R171"
+		(property "Reference" "R71"
 			(at 134.874 78.994 90)
 			(effects
@@
 			(project "Project-Star"
 				(path "/fc8533bc-25dd-4c20-9b4c-ffebebd6739b/e8da5d81-614b-4fe5-84b3-4c351fab7114/e3d465d4-4bae-42f2-91c8-f61f15aa6ae9"
-					(reference "R171")
-					(unit 1)
-				)
+					(reference "R71")
+					(unit 1)
+				)
