File: High Voltage REGSRC Supply.kicad_sch (KiCad schematic)
At the start: 10 parts, among them Q16 BSS123

Commit message: ready to start first pass review on bms
Parts:
- renumbered C31 to C30, C32 to C31, C33 to C32, C34 to C33, D29 to D32, Q16 to Q17, R71 to R67, R72 to R68, R73 to R69, R74 to R70
