File: MCU Current Sense.kicad_sch (KiCad schematic)
At the start: 5 parts, among them Q21 CSD23381F4

Commit message: worked on MCU
Parts:
- renumbered Q21 to Q9, R101 to R44, R102 to R45, R103 to R46, R110 to R47
Changed lines of the file:
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@@
 		(on_board yes)
 		(dnp no)
-		(property "Reference" "Q21"
+		(property "Reference" "Q9"
 			(at 149.86 74.93 0)
 			(effects
@@
 			(project "Project-Star"
 				(path "/fc8533bc-25dd-4c20-9b4c-ffebebd6739b/e8da5d81-614b-4fe5-84b3-4c351fab7114/0284ed28-c434-46ce-a359-08e3f2d412cf"
-					(reference "Q21")
+					(reference "Q9")
 					(unit 1)
 				)
@@
 		(on_board yes)
 		(dnp no)
-		(property "Reference" "R103"
+		(property "Reference" "R46"
 			(at 151.892 101.854 0)
 			(effects
@@
 			(project "Project-Star"
 				(path "/fc8533bc-25dd-4c20-9b4c-ffebebd6739b/e8da5d81-614b-4fe5-84b3-4c351fab7114/0284ed28-c434-46ce-a359-08e3f2d412cf"
-					(reference "R103")
+					(reference "R46")
 					(unit 1)
 				)
@@
 		(on_board yes)
 		(dnp no)
-		(property "Reference" "R110"
+		(property "Reference" "R47"
 			(at 155.702 96.52 90)
 			(effects
@@
 			(project "Project-Star"
 				(path "/fc8533bc-25dd-4c20-9b4c-ffebebd6739b/e8da5d81-614b-4fe5-84b3-4c351fab7114/0284ed28-c434-46ce-a359-08e3f2d412cf"
-					(reference "R110")
+					(reference "R47")
 					(unit 1)
 				)
@@
 		(on_board yes)
 		(dnp no)
-		(property "Reference" "R101"
+		(property "Reference" "R44"
 			(at 136.398 96.774 90)
 			(effects
@@
 			(project "Project-Star"
 				(path "/fc8533bc-25dd-4c20-9b4c-ffebebd6739b/e8da5d81-614b-4fe5-84b3-4c351fab7114/0284ed28-c434-46ce-a359-08e3f2d412cf"
-					(reference "R101")
+					(reference "R44")
 					(unit 1)
 				)
@@
 		(on_board yes)
 		(dnp no)
-		(property "Reference" "#PWR049"
+		(property "Reference" "#PWR07"
 			(at 149.86 116.84 0)
 			(effects
@@
 			(project "Project-Star"
 				(path "/fc8533bc-25dd-4c20-9b4c-ffebebd6739b/e8da5d81-614b-4fe5-84b3-4c351fab7114/0284ed28-c434-46ce-a359-08e3f2d412cf"
-					(reference "#PWR049")
+					(reference "#PWR07")
 					(unit 1)
 				)
@@
 		(on_board yes)
 		(dnp no)
-		(property "Reference" "R102"
+		(property "Reference" "R45"
 			(at 151.892 86.614 0)
 			(effects
@@
 			(project "Project-Star"
 				(path "/fc8533bc-25dd-4c20-9b4c-ffebebd6739b/e8da5d81-614b-4fe5-84b3-4c351fab7114/0284ed28-c434-46ce-a359-08e3f2d412cf"
-					(reference "R102")
-					(unit 1)
-				)
+					(reference "R45")
+					(unit 1)
+				)
