File: Passive Balancing Circuit.kicad_sch (KiCad schematic)
At the start: 70 parts, among them Q13 DMN2004K, Q14 DMN2004K, Q38 DMN2004K, Q39 DMN2004K, Q40 DMN2004K, Q41 DMN2004K, Q42 DMN2004K, Q43 DMN2004K

Commit message: worked on MCU
Parts:
- renumbered C31 to C1, C71 to C10, C32 to C2, C33 to C3, C34 to C4, C36 to C5, C37 to C6, C38 to C7, C69 to C8, C70 to C9, D24 to D1, D64 to D10, D65 to D11, D66 to D12, D67 to D13, D68 to D14, D69 to D15, D70 to D16, D71 to D17, D25 to D2, D26 to D3, D35 to D4, D59 to D5, D60 to D6, D61 to D7, D62 to D8, D63 to D9, Q13 to Q1, Q14 to Q2, Q38 to Q3, Q39 to Q4, Q40 to Q5, Q41 to Q6, Q42 to Q7, Q43 to Q8, R36 to R1, R186 to R10, R187 to R11, R188 to R12, R189 to R13, R190 to R14, R191 to R15, R193 to R16, R194 to R17, R195 to R18, R196 to R19, R59 to R2, R197 to R20, R198 to R21, R199 to R22, R200 to R23, R201 to R24, R202 to R25, R203 to R26, R204 to R27, R205 to R28, R206 to R29, R60 to R3, R207 to R30, R208 to R31, R209 to R32, R210 to R33, R211 to R34, R212 to R35, R61 to R4, R62 to R5, R63 to R6, R64 to R7, R65 to R8, R82 to R9
