File: Passive Balancing Circuit.kicad_sch (KiCad schematic)
At the start: 70 parts, among them Q1 DMN2004K, Q2 DMN2004K, Q3 DMN2004K, Q4 DMN2004K, Q5 DMN2004K, Q6 DMN2004K, Q7 DMN2004K, Q8 DMN2004K

Commit message: ready to start first pass review on bms
Parts:
- D1, D2, D3, D4, D5, D6, D7, D8: value LED -> RED
