File: Wake Up.kicad_sch (KiCad schematic)
At the start: 12 parts, among them Q10 ZXMP10A13F, Q18 BSS123, Q23 BSS123

Commit message: ready to start first pass review on bms
Parts:
- removed R51: 51k, symbol Device:R
- added R56, R57: 100k, symbol Device:R
- D30: renamed from D25; value 3V9 -> 3V3
- renumbered C19 to C23, D24 to D28, D23 to D29, Q23 to Q14, Q10 to Q15, Q18 to Q16, R48 to R55, R49 to R58, R50 to R59, R52 to R60
Connections:
- net at Q14.2 (S): now also R56.1, R57.1
- net WAKE: no longer names the net of D28.2 (A), D30.1 (K)
- net WAKE: now also R56.2, R57.2
Other:
- note removed: "***TODO: Figure out what to do with the possibly exposed "WAKE"***"
- moved on the sheet: D28, R60
