File: Fuel Gauge.kicad_sch (KiCad schematic)
At the start: 32 parts, among them Q18 ZXMP10A13F, Q19 BSS123, Q20 BCX56, U3 BQ78350DBT-R1A, U4 TPD1E05U06DYA, U5 TPD1E05U06DYA

Commit message: I still need to add the 6V line and test points
Other:
- note added: "Fuel Gauge"
Changed lines of the file:
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@@
 	(generator_version "9.0")
 	(paper "A4")
+	(text "Fuel Gauge"
+		(exclude_from_sim no)
+		(at 152.654 49.784 0)
+		(effects
+			(font
+				(size 6.35 6.35)
+				(thickness 1.27)
+				(bold yes)
+			)
+		)
+	)
 	(text "from TIDA-00792"
 		(exclude_from_sim no)
