File: BMS Protection Board.kicad_sch (KiCad schematic)
At the start: 0 parts

Commit message: in progress still
Changed lines of the file:
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@@
 		(color 0 0 0 0)
 	)
-	(wire
-		(pts
-			(xy 217.17 26.67) (xy 246.38 26.67)
+	(junction
+		(at 237.49 26.67)
+		(diameter 0)
+		(color 0 0 0 0)
+	)
+	(wire
+		(pts
+			(xy 217.17 26.67) (xy 237.49 26.67)
 		)
 		(stroke
@@
 	(wire
 		(pts
+			(xy 139.7 59.69) (xy 158.75 59.69)
+		)
+		(stroke
+			(width 0)
+			(type default)
+		)
+	)
+	(wire
+		(pts
 			(xy 82.55 111.76) (xy 71.12 111.76)
 		)
@@
 	(wire
 		(pts
+			(xy 139.7 15.24) (xy 237.49 15.24)
+		)
+		(stroke
+			(width 0)
+			(type default)
+		)
+	)
+	(wire
+		(pts
 			(xy 110.49 143.51) (xy 124.46 143.51)
 		)
@@
 	(wire
 		(pts
+			(xy 237.49 26.67) (xy 246.38 26.67)
+		)
+		(stroke
+			(width 0)
+			(type default)
+		)
+	)
+	(wire
+		(pts
 			(xy 96.52 143.51) (xy 102.87 143.51)
 		)
@@
 	(wire
 		(pts
-			(xy 158.75 71.12) (xy 146.05 71.12)
+			(xy 130.81 58.42) (xy 22.86 58.42)
 		)
 		(stroke
@@
 	(wire
 		(pts
-			(xy 151.13 59.69) (xy 158.75 59.69)
-		)
-		(stroke
-			(width 0)
-			(type default)
-		)
-	)
-	(wire
-		(pts
 			(xy 27.94 123.19) (xy 35.56 123.19)
 		)
@@
 	(wire
 		(pts
+			(xy 22.86 58.42) (xy 22.86 69.85)
+		)
+		(stroke
+			(width 0)
+			(type default)
+		)
+	)
+	(wire
+		(pts
 			(xy 16.51 86.36) (xy 39.37 86.36)
 		)
@@
 	(wire
 		(pts
+			(xy 237.49 15.24) (xy 237.49 26.67)
+		)
+		(stroke
+			(width 0)
+			(type default)
+		)
+	)
+	(wire
+		(pts
 			(xy 110.49 148.59) (xy 124.46 148.59)
 		)
@@
 	(wire
 		(pts
+			(xy 130.81 71.12) (xy 130.81 58.42)
+		)
+		(stroke
+			(width 0)
+			(type default)
+		)
+	)
+	(wire
+		(pts
 			(xy 64.77 74.93) (xy 88.9 74.93)
 		)
@@
 	(wire
 		(pts
+			(xy 139.7 59.69) (xy 139.7 15.24)
+		)
+		(stroke
+			(width 0)
+			(type default)
+		)
+	)
+	(wire
+		(pts
 			(xy 30.48 140.97) (xy 46.99 140.97)
 		)
@@
 	(wire
 		(pts
-			(xy 39.37 69.85) (xy 27.94 69.85)
+			(xy 130.81 71.12) (xy 158.75 71.12)
 		)
 		(stroke
@@
 		)
 		(stroke
+			(width 0)
+			(type default)
+		)
+	)
+	(wire
+		(pts
+			(xy 22.86 69.85) (xy 39.37 69.85)
+		)
+		(stroke
