File: Charger FET Array.kicad_sch (KiCad schematic)
At the start: 32 parts, among them J9 To Battery Pack, Q21 CSD19531Q5A, Q22 CSD19531Q5A, Q23 CSD19531Q5A, Q24 CSD19531Q5A

Commit message: in progress still
Parts:
- removed J9: To Battery Pack, symbol Connector_Generic:Conn_01x03
Other:
- note added: "we need to find what to put for this based off what we can buy more uH is better, less Ω is better"
- note removed: "we need to find what to put for this based off what we can buy"
Changed lines of the file:
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@@
 		)
 	)
-	(text "we need to find what to put \nfor this based off what we can buy"
+	(text "we need to find what to put \nfor this based off what we can buy\nmore uH is better, less Ω is better"
 		(exclude_from_sim no)
-		(at 140.97 101.346 0)
+		(at 140.716 100.076 0)
 		(effects
 			(font
@@
 	)
 	(junction
-		(at 229.87 116.84)
-		(diameter 0)
-		(color 0 0 0 0)
-	)
-	(junction
 		(at 53.34 105.41)
 		(diameter 0)
@@
 	)
 	(junction
-		(at 242.57 83.82)
-		(diameter 0)
-		(color 0 0 0 0)
-	)
-	(junction
 		(at 80.01 83.82)
 		(diameter 0)
@@
 	(wire
 		(pts
-			(xy 251.46 88.9) (xy 248.92 88.9)
-		)
-		(stroke
-			(width 0)
-			(type default)
-		)
-	)
-	(wire
-		(pts
 			(xy 115.57 107.95) (xy 115.57 99.06)
 		)
@@
 	(wire
 		(pts
-			(xy 242.57 80.01) (xy 242.57 83.82)
-		)
-		(stroke
-			(width 0)
-			(type default)
-		)
-	)
-	(wire
-		(pts
 			(xy 71.12 107.95) (xy 71.12 105.41)
 		)
@@
 	(wire
 		(pts
-			(xy 229.87 116.84) (xy 248.92 116.84)
-		)
-		(stroke
-			(width 0)
-			(type default)
-		)
-	)
-	(wire
-		(pts
 			(xy 229.87 87.63) (xy 229.87 83.82)
 		)
@@
 	(wire
 		(pts
-			(xy 229.87 83.82) (xy 242.57 83.82)
+			(xy 229.87 83.82) (xy 241.3 83.82)
 		)
 		(stroke
@@
 	(wire
 		(pts
-			(xy 245.11 86.36) (xy 251.46 86.36)
-		)
-		(stroke
-			(width 0)
-			(type default)
-		)
-	)
-	(wire
-		(pts
 			(xy 212.09 83.82) (xy 217.17 83.82)
 		)
@@
 	(wire
 		(pts
-			(xy 248.92 88.9) (xy 248.92 116.84)
-		)
-		(stroke
-			(width 0)
-			(type default)
-		)
-	)
-	(wire
-		(pts
 			(xy 66.04 83.82) (xy 71.12 83.82)
 		)
@@
 	(wire
 		(pts
-			(xy 234.95 80.01) (xy 242.57 80.01)
-		)
-		(stroke
-			(width 0)
-			(type default)
-		)
-	)
-	(wire
-		(pts
 			(xy 224.79 99.06) (xy 229.87 99.06)
 		)
@@
 		(pts
 			(xy 33.02 137.16) (xy 41.91 137.16)
-		)
-		(stroke
-			(width 0)
-			(type default)
-		)
-	)
-	(wire
-		(pts
-			(xy 242.57 83.82) (xy 251.46 83.82)
 		)
 		(stroke
@@
 		)
 	)
-	(label "TS"
-		(at 248.92 86.36 0)
-		(effects
-			(font
-				(size 1.27 1.27)
-			)
-			(justify left bottom)
-		)
-	)
 	(label "SW1"
 		(at 99.06 107.95 0)
@@
 	)
 	(label "PACK+"
-		(at 242.57 80.01 180)
+		(at 241.3 83.82 180)
 		(effects
 			(font
@@
 	(hierarchical_label "PACK+"
 		(shape bidirectional)
-		(at 234.95 80.01 180)
-		(effects
-			(font
-				(size 1.27 1.27)
-			)
-			(justify right)
+		(at 241.3 83.82 0)
+		(effects
+			(font
+				(size 1.27 1.27)
+			)
+			(justify left)
 		)
 	)
@@
 			)
 			(justify left)
-		)
-	)
-	(hierarchical_label "TS"
-		(shape output)
-		(at 245.11 86.36 180)
-		(effects
-			(font
-				(size 1.27 1.27)
-			)
-			(justify right)
 		)
 	)
@@
 					(unit 1)
 				)
-			)
-		)
-	)
-	(symbol
-		(lib_id "Connector_Generic:Conn_01x03")
-		(at 256.54 86.36 0)
-		(unit 1)
-		(exclude_from_sim no)
-		(in_bom yes)
-		(on_board yes)
-		(dnp no)
-		(fields_autoplaced yes)
-		(property "Reference" "J9"
-			(at 259.08 85.0899 0)
-			(effects
-				(font
-					(size 1.27 1.27)
-				)
-				(justify left)
-			)
-		)
-		(property "Value" "To Battery Pack"
-			(at 259.08 87.6299 0)
-			(effects
-				(font
-					(size 1.27 1.27)
-				)
-				(justify left)
-			)
-		)
-		(property "Footprint" ""
-			(at 256.54 86.36 0)
-			(effects
-				(font
-					(size 1.27 1.27)
-				)
-				(hide yes)
-			)
-		)
-		(property "Datasheet" "~"
-			(at 256.54 86.36 0)
-			(effects
-				(font
-					(size 1.27 1.27)
-				)
-				(hide yes)
-			)
-		)
-		(property "Description" "Generic connector, single row, 01x03, script generated (kicad-library-utils/schlib/autogen/connector/)"
-			(at 256.54 86.36 0)
-			(effects
-				(font
-					(size 1.27 1.27)
-				)
-				(hide yes)
-			)
-		)
-		(pin "1"
-		)
-		(pin "3"
-		)
-		(pin "2"
-		)
-		(instances
-			(project ""
-				(path "/fc8533bc-25dd-4c20-9b4c-ffebebd6739b/ec72a35b-e7f2-4422-8859-60e9fb848154/9fb42b36-af5a-430a-ae71-09fe6d8fbe9c"
-					(reference "J9")
-					(unit 1)
-				)
