File: Pack Switching and Current Sensing.kicad_sch (KiCad schematic)
At the start: 30 parts, among them Q10 CSD19531Q5A, Q11 ZXMP10A13F, Q12 CSD19531Q5A, Q13 CSD19531Q5A, Q9 CSD19531Q5A

Commit message: in progress still
Parts:
- added R131: 10M, symbol Device:R
Connections:
- net PCHG: now also R131.1
- net at Q10.5 (D), Q11.2 (S), Q12.5 (D)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: now also R131.2
Other:
- moved on the sheet: C19, C20, C21, C22, D23, D24, D25, D26, D27, E1, FB1, FB2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
