File: USB-C 5V Buck.kicad_sch (KiCad schematic)
At the start: 27 parts, among them Q25 CSD19531Q5A, Q26 CSD19531Q5A, U12 LM5148RGYR, U8 TPSM365R3RDNR

Commit message: in progress still
Parts:
- removed C46: 1u, symbol Device:C
- removed C47: 100n, symbol Device:C
- removed C48: 2u2, symbol Device:C
- removed C49, C50: 22u, symbol Device:C
- removed C51: 10p, symbol Device:C
- removed R88: 19k6, symbol Device:R
- removed R89: 40k2, symbol Device:R
- removed R90: 10k, symbol Device:R
- removed U8: TPSM365R3RDNR, QFN-FCMOD_365R6FRDN_TEX, symbol TPSM365R3RDNR:TPSM365R3RDNR
Connections:
- no-connect marks 7 -> 5
Other:
- note added: "5V, 5A Line"
- note added: "P5V0 must support 3A(VBUS) + 0.315A(VCONN) = 3.315A with headroom, 5A is a good amount"
- note removed: "This is what they put in PMP41062, but it seems wrong? This provides a Imax of 300mA However, P5V0 must support 3A(VBUS) + 0.315A(VCONN) = 3.315A with headroom, 5A is a good amount"
