File: USB-C PD Controller.kicad_sch (KiCad schematic)
At the start: 20 parts, among them U10 TPS25751DREFR

Commit message: in progress still
Changed lines of the file:
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@@
-	)
-	(junction
-		(at 80.01 80.01)
-		(diameter 0)
-		(color 0 0 0 0)
 	)
 	(junction
@@
 		(pts
 			(xy 110.49 120.65) (xy 107.95 120.65)
-		)
-		(stroke
-			(width 0)
-			(type default)
-		)
-	)
-	(wire
-		(pts
-			(xy 76.2 80.01) (xy 80.01 80.01)
 		)
 		(stroke
@@
 		)
 	)
-	(hierarchical_label "LDO_1V5"
-		(shape output)
-		(at 76.2 80.01 180)
-		(effects
-			(font
-				(size 1.27 1.27)
-			)
-			(justify right)
-		)
-	)
 	(hierarchical_label "C_CC2"
 		(shape output)
@@
 	)
 	(hierarchical_label "PPHV"
-		(shape input)
+		(shape bidirectional)
 		(at 99.06 127 180)
 		(effects
