File: USB-C Power Delivery.kicad_sch (KiCad schematic)
At the start: 0 parts

Commit message: in progress still
Other:
- sheet Buck-Boost Charger ports: added none; removed BTST1, BTST2, DRV_SUP, FB, FBG, FSW_SYNC, ICHG, ILIM_HIZ, REGN, STAT1, STAT2, TS, ~{CE}, ~{INT}, ~{PG}
- sheet Charger FET Array ports: added none; removed TS
- sheet USB-C PD Controller ports: added none; removed LDO_1V5
Changed lines of the file:
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@@
+	)
+	(junction
+		(at 130.81 67.31)
+		(diameter 0)
+		(color 0 0 0 0)
 	)
 	(junction
@@
 		(color 0 0 0 0)
 	)
+	(junction
+		(at 130.81 34.29)
+		(diameter 0)
+		(color 0 0 0 0)
+	)
 	(wire
 		(pts
@@
 	(wire
 		(pts
+			(xy 130.81 88.9) (xy 163.83 88.9)
+		)
+		(stroke
+			(width 0)
+			(type default)
+		)
+	)
+	(wire
+		(pts
 			(xy 217.17 43.18) (xy 224.79 43.18)
 		)
@@
 	(wire
 		(pts
+			(xy 130.81 34.29) (xy 133.35 34.29)
+		)
+		(stroke
+			(width 0)
+			(type default)
+		)
+	)
+	(wire
+		(pts
 			(xy 71.12 69.85) (xy 71.12 43.18)
 		)
@@
 	(wire
 		(pts
-			(xy 198.12 86.36) (xy 224.79 86.36)
-		)
-		(stroke
-			(width 0)
-			(type default)
-		)
-	)
-	(wire
-		(pts
 			(xy 114.3 45.72) (xy 128.27 45.72)
 		)
@@
 		(pts
 			(xy 114.3 38.1) (xy 128.27 38.1)
+		)
+		(stroke
+			(width 0)
+			(type default)
+		)
+	)
+	(wire
+		(pts
+			(xy 130.81 88.9) (xy 130.81 67.31)
 		)
 		(stroke
@@
 	(label "LODRV2"
 		(at 208.28 73.66 0)
-		(effects
-			(font
-				(size 1.27 1.27)
-			)
-			(justify left bottom)
-		)
-	)
-	(label "TS"
-		(at 208.28 86.36 0)
 		(effects
 			(font
@@
 			)
 			(justify right)
+		)
+	)
+	(hierarchical_label "SDA"
+		(shape output)
+		(at 148.59 40.64 180)
+		(effects
+			(font
+				(size 1.27 1.27)
+			)
+			(justify right)
+		)
+	)
+	(hierarchical_label "SCL"
+		(shape output)
+		(at 148.59 38.1 180)
+		(effects
+			(font
+				(size 1.27 1.27)
+			)
+			(justify right)
+		)
+	)
+	(hierarchical_label "LDO_3V3"
+		(shape output)
+		(at 133.35 34.29 0)
+		(effects
+			(font
+				(size 1.27 1.27)
+			)
+			(justify left)
 		)
 	)
@@
 			)
 		)
-		(pin "STAT2" input
-			(at 163.83 43.18 180)
-			(effects
-				(font
-					(size 1.27 1.27)
-				)
-				(justify left)
-			)
-		)
-		(pin "TS" input
-			(at 198.12 86.36 0)
-			(effects
-				(font
-					(size 1.27 1.27)
-				)
-				(justify right)
-			)
-		)
 		(pin "P_OUT" input
 			(at 198.12 88.9 0)
@@
 			)
 		)
-		(pin "~{INT}" output
-			(at 163.83 55.88 180)
-			(effects
-				(font
-					(size 1.27 1.27)
-				)
-				(justify left)
-			)
-		)
-		(pin "STAT1" input
-			(at 163.83 58.42 180)
-			(effects
-				(font
-					(size 1.27 1.27)
-				)
-				(justify left)
-			)
-		)
-		(pin "BTST1" passive
-			(at 163.83 60.96 180)
-			(effects
-				(font
-					(size 1.27 1.27)
-				)
-				(justify left)
-			)
-		)
-		(pin "~{CE}" passive
-			(at 163.83 63.5 180)
-			(effects
-				(font
-					(size 1.27 1.27)
-				)
-				(justify left)
-			)
-		)
-		(pin "REGN" output
-			(at 163.83 66.04 180)
-			(effects
-				(font
-					(size 1.27 1.27)
-				)
-				(justify left)
-			)
-		)
 		(pin "ACUV" input
 			(at 198.12 63.5 0)
@@
 			)
 		)
-		(pin "ILIM_HIZ" passive
-			(at 163.83 71.12 180)
-			(effects
-				(font
-					(size 1.27 1.27)
-				)
-				(justify left)
-			)
-		)
 		(pin "SRP" input
 			(at 198.12 76.2 0)
@@
 			)
 		)
-		(pin "ICHG" passive
-			(at 163.83 78.74 180)
-			(effects
-				(font
-					(size 1.27 1.27)
-				)
-				(justify left)
-			)
-		)
 		(pin "HIDRV2" input
 			(at 198.12 68.58 0)
@@
 			)
 		)
-		(pin "FSW_SYNC" passive
-			(at 163.83 91.44 180)
-			(effects
-				(font
-					(size 1.27 1.27)
-				)
-				(justify left)
-			)
-		)
-		(pin "FBG" passive
-			(at 163.83 93.98 180)
-			(effects
-				(font
-					(size 1.27 1.27)
-				)
-				(justify left)
-			)
-		)
 		(pin "HIDRV1" input
 			(at 198.12 66.04 0)
@@
 			)
 		)
-		(pin "BTST2" passive
-			(at 198.12 36.83 0)
-			(effects
-				(font
-					(size 1.27 1.27)
-				)
-				(justify right)
-			)
-		)
-		(pin "~{PG}" output
-			(at 198.12 39.37 0)
-			(effects
-				(font
-					(size 1.27 1.27)
-				)
-				(justify right)
-			)
-		)
 		(pin "SRN" input
 			(at 198.12 78.74 0)
-			(effects
-				(font
-					(size 1.27 1.27)
-				)
-				(justify right)
-			)
-		)
-		(pin "FB" passive
-			(at 198.12 41.91 0)
-			(effects
-				(font
-					(size 1.27 1.27)
-				)
-				(justify right)
-			)
-		)
-		(pin "DRV_SUP" input
-			(at 198.12 44.45 0)
 			(effects
 				(font
@@
 			)
 		)
-		(pin "TS" output
-			(at 224.79 86.36 180)
-			(effects
-				(font
-					(size 1.27 1.27)
-				)
-				(justify left)
-			)
-		)
 		(pin "VSYS" output
 			(at 224.79 93.98 180)
@@
 			)
 		)
-		(pin "LDO_1V5" output
-			(at 114.3 31.75 0)
-			(effects
-				(font
-					(size 1.27 1.27)
-				)
-				(justify right)
-			)
-		)
 		(pin "C_CC2" output
 			(at 114.3 40.64 0)
@@
 			)
 		)
-		(pin "PPHV" input
+		(pin "PPHV" bidirectional
 			(at 78.74 34.29 180)
 			(effects
