File: old-revision/20V_Power_Line.kicad_sch (KiCad schematic)
At the start: 42 parts, among them CN1 SC In, CN2 SC Out, Q1 CSD18543Q3A, Q2 CSD18543Q3A, U3 TP Vin, U4 LM25145RGYR, U5 TP GND, U6 TP Vout

Commit message: current progress
Parts:
- removed Ccomp2: 100p, easyeda2kicad:C0402, symbol easyeda2kicad:0402CG101J500NT
- removed Css1: 39n, easyeda2kicad:C0603, symbol easyeda2kicad:0603B393K500NT
- added Ccomp2: 110p, easyeda2kicad:C0402, symbol easyeda2kicad:GRM1555C1H111JA01D
- added Css1: 150n, easyeda2kicad:C0603, symbol easyeda2kicad:0603B154K500NT
Connections:
- net GND: now also Css1.2
- net at U4.3 (SS/TRK): now also Css1.1
- net at Ccomp1.1, U4.4 (COMP): now also Ccomp2.1
- net at Ccomp3.2, Rcomp1.2, Rfb1.2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: now also Ccomp2.2
