File: old-revision/Project-Star.kicad_pcb (KiCad board)
At the start: 4 copper layers, 54.5 x 29.8 mm, 42 parts, among them CN1 SC In, CN2 SC Out, Q1 CSD18543Q3A, Q2 CSD18543Q3A, U4 LM25145RGYR

Commit message: current progress
Parts:
- Ccomp2: value 100p -> 110p
- Css1: value 39n -> 150n
- moved VOUT 34.1 mm to (182.8, 97.3), turned to 0 degrees
- moved GND 26.5 mm to (182.3, 92.0), turned to 0 degrees
- moved H1 4.70 mm to (169.2, 111.9)
- moved VIN 0.22 mm to (131.3, 95.9), turned to 0 degrees
- moved H2 0.10 mm to (122.4, 111.8)
Changed lines of the file:
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@@
 	(footprint "PCM_SL_Mechanical:MountingHole_3.2mm_Pad"
 		(layer "F.Cu")
-		(at 122.5 111.8 180)
+		(at 122.4 111.8 180)
 		(property "Reference" "H2"
 			(at 0 -4.064 180)
@@
 		(embedded_fonts no)
 	)
+	(footprint "easyeda2kicad:TEST-TH_BD3.17-P1.87"
+		(layer "F.Cu")
+		(at 182.3 92)
+		(property "Reference" "GND"
+			(at 2.2 -2.5 0)
+			(unlocked yes)
+			(layer "F.SilkS")
+			(effects
+				(font
+					(size 1 1)
+					(thickness 0.15)
+				)
+			)
+		)
+		(property "Value" "TP GND"
+			(at 0 4 0)
+			(unlocked yes)
+			(layer "F.Fab")
+			(effects
+				(font
+					(size 1 1)
+					(thickness 0.15)
+				)
+			)
+		)
+		(property "Datasheet" "https://lcsc.com/product-detail/Test-Points-Test-Rings_Keystone_5011_Keystone-5011_C238127.html"
+			(at 0 0 0)
+			(unlocked yes)
+			(layer "F.Fab")
+			(hide yes)
+			(effects
+				(font
+					(size 1 1)
+					(thickness 0.15)
+				)
+			)
+		)
+		(property "Description" ""
+			(at 0 0 0)
+			(unlocked yes)
+			(layer "F.Fab")
+			(hide yes)
+			(effects
+				(font
+					(size 1 1)
+					(thickness 0.15)
+				)
+			)
+		)
+		(property "LCSC Part" "C238127"
+			(at 0 0 0)
+			(unlocked yes)
+			(layer "F.Fab")
+			(hide yes)
+			(effects
+				(font
+					(size 1 1)
+					(thickness 0.15)
+				)
+			)
+		)
+		(sheetname "/20V_Power_Line/")
+		(sheetfile "20V_Power_Line.kicad_sch")
+		(attr through_hole)
+		(fp_circle
+			(center 0 0)
+			(end 1.6 0)
+			(stroke
+				(width 0.1)
+				(type solid)
+			)
+			(fill no)
+			(layer "F.SilkS")
+		)
+		(fp_circle
+			(center 0 0)
+			(end 0.42 0)
+			(stroke
+				(width 0.1)
+				(type solid)
+			)
+			(fill no)
+			(layer "F.Fab")
+		)
+		(fp_circle
+			(center 1.73 -1.73)
+			(end 1.76 -1.73)
+			(stroke
+				(width 0.1)
+				(type solid)
+			)
+			(fill no)
+			(layer "F.Fab")
+		)
+		(fp_text user "${REFERENCE}"
+			(at 0 0 0)
+			(unlocked yes)
+			(layer "F.Fab")
+			(effects
+				(font
+					(size 1 1)
+					(thickness 0.15)
+				)
+			)
+		)
+		(pad "1" thru_hole circle
+			(at 0 0)
+			(size 2.7 2.7)
+			(drill 1.869999)
+			(layers "*.Cu" "*.Mask")
+			(remove_unused_layers no)
+			(net 19 "GND")
+			(pinfunction "1")
+			(pintype "unspecified")
+		)
+		(embedded_fonts no)
+		(model "${EASYEDA2KICAD}/easyeda2kicad.3dshapes/TEST-TH_BD3.17-P1.87.wrl"
+			(offset
+				(xyz -0.02 -0 0)
+			)
+			(scale
+				(xyz 1 1 1)
+			)
+			(rotate
+				(xyz 0 0 0)
+			)
+		)
+	)
 	(footprint "easyeda2kicad:VSONP-8_L3.1-W3.1-P0.65-LS3.5-BL"
 		(layer "F.Cu")
@@
 	(footprint "easyeda2kicad:TEST-TH_BD3.17-P1.87"
 		(layer "F.Cu")
-		(at 155.79 92.75 90)
-		(property "Reference" "GND"
-			(at 0 -2.54 90)
+		(at 131.3 95.9)
+		(property "Reference" "VIN"
+			(at -0.3 -2.4 0)
 			(unlocked yes)
 			(layer "F.SilkS")
@@
 			)
 		)
-		(property "Value" "TP GND"
-			(at 0 4 90)
+		(property "Value" "TP Vin"
+			(at 0 4 0)
 			(unlocked yes)
 			(layer "F.Fab")
@@
 		)
 		(property "Datasheet" "https://lcsc.com/product-detail/Test-Points-Test-Rings_Keystone_5011_Keystone-5011_C238127.html"
-			(at 0 0 90)
+			(at 0 0 0)
 			(unlocked yes)
 			(layer "F.Fab")
@@
 		)
 		(property "Description" ""
-			(at 0 0 90)
+			(at 0 0 0)
 			(unlocked yes)
 			(layer "F.Fab")
@@
 		)
 		(property "LCSC Part" "C238127"
-			(at 0 0 90)
+			(at 0 0 0)
 			(unlocked yes)
 			(layer "F.Fab")
@@
 		)
 		(fp_circle
-			(center 1.73 -1.73)
-			(end 1.76 -1.73)
+			(center 0 0)
+			(end 0.42 0)
 			(stroke
 				(width 0.1)
@@
 		)
 		(fp_circle
-			(center 0 0)
-			(end 0.42 0)
+			(center 1.73 -1.73)
+			(end 1.76 -1.73)
 			(stroke
 				(width 0.1)
@@
 		)
 		(fp_text user "${REFERENCE}"
-			(at 0 0 90)
+			(at 0 0 0)
 			(unlocked yes)
 			(layer "F.Fab")
@@
 		)
 		(pad "1" thru_hole circle
-			(at 0 0 90)
+			(at 0 0)
 			(size 2.7 2.7)
 			(drill 1.869999)
 			(layers "*.Cu" "*.Mask")
 			(remove_unused_layers no)
-			(net 19 "GND")
+			(net 4 "/20V_Power_Line/Vin")
 			(pinfunction "1")
 			(pintype "unspecified")
@@
 	(footprint "easyeda2kicad:TEST-TH_BD3.17-P1.87"
 		(layer "F.Cu")
-		(at 152 112 90)
+		(at 182.8 97.3)
 		(property "Reference" "VOUT"
-			(at -2.5 0 0)
+			(at 3.7 1.4 0)
 			(unlocked yes)
 			(layer "F.SilkS")
@@
 		)
 		(property "Value" "TP Vout"
-			(at 0 4 90)
+			(at 0 4 0)
 			(unlocked yes)
 			(layer "F.Fab")
@@
 		)
 		(property "Datasheet" "https://lcsc.com/product-detail/Test-Points-Test-Rings_Keystone_5011_Keystone-5011_C238127.html"
-			(at 0 0 90)
+			(at 0 0 0)
 			(unlocked yes)
 			(layer "F.Fab")
@@
 		)
 		(property "Description" ""
-			(at 0 0 90)
+			(at 0 0 0)
 			(unlocked yes)
 			(layer "F.Fab")
@@
 		)
 		(property "LCSC Part" "C238127"
-			(at 0 0 90)
+			(at 0 0 0)
 			(unlocked yes)
 			(layer "F.Fab")
@@
 		)
 		(fp_circle
-			(center 1.73 -1.73)
-			(end 1.76 -1.73)
-			(stroke
-				(width 0.1)
-				(type solid)
-			)
-			(fill no)
-			(layer "F.Fab")
-		)
-		(fp_circle
 			(center 0 0)
 			(end 0.42 0)
@@
 			(layer "F.Fab")
 		)
-		(fp_text user "${REFERENCE}"
-			(at 0 0 90)
-			(unlocked yes)
-			(layer "F.Fab")
-			(effects
-				(font
-					(size 1 1)
-					(thickness 0.15)
-				)
-			)
-		)
-		(pad "1" thru_hole circle
-			(at 0 0 90)
-			(size 2.7 2.7)
-			(drill 1.869999)
-			(layers "*.Cu" "*.Mask")
-			(remove_unused_layers no)
-			(net 11 "/20V_Power_Line/Vout")
-			(pinfunction "1")
-			(pintype "unspecified")
-		)
-		(embedded_fonts no)
-		(model "${EASYEDA2KICAD}/easyeda2kicad.3dshapes/TEST-TH_BD3.17-P1.87.wrl"
-			(offset
-				(xyz -0.02 -0 0)
-			)
-			(scale
-				(xyz 1 1 1)
-			)
-			(rotate
-				(xyz 0 0 0)
-			)
-		)
-	)
-	(footprint "easyeda2kicad:TEST-TH_BD3.17-P1.87"
-		(layer "F.Cu")
-		(at 131.5 96 90)
-		(property "Reference" "VIN"
-			(at 2.5 -0.75 0)
-			(unlocked yes)
-			(layer "F.SilkS")
-			(effects
-				(font
-					(size 1 1)
-					(thickness 0.15)
-				)
-			)
-		)
-		(property "Value" "TP Vin"
-			(at 0 4 90)
-			(unlocked yes)
-			(layer "F.Fab")
-			(effects
-				(font
-					(size 1 1)
-					(thickness 0.15)
-				)
-			)
-		)
-		(property "Datasheet" "https://lcsc.com/product-detail/Test-Points-Test-Rings_Keystone_5011_Keystone-5011_C238127.html"
-			(at 0 0 90)
-			(unlocked yes)
-			(layer "F.Fab")
-			(hide yes)
-			(effects
-				(font
-					(size 1 1)
-					(thickness 0.15)
-				)
-			)
-		)
-		(property "Description" ""
-			(at 0 0 90)
-			(unlocked yes)
-			(layer "F.Fab")
-			(hide yes)
-			(effects
-				(font
-					(size 1 1)
-					(thickness 0.15)
-				)
-			)
-		)
-		(property "LCSC Part" "C238127"
-			(at 0 0 90)
-			(unlocked yes)
-			(layer "F.Fab")
-			(hide yes)
-			(effects
-				(font
-					(size 1 1)
-					(thickness 0.15)
-				)
-			)
-		)
-		(sheetname "/20V_Power_Line/")
-		(sheetfile "20V_Power_Line.kicad_sch")
-		(attr through_hole)
-		(fp_circle
-			(center 0 0)
-			(end 1.6 0)
-			(stroke
-				(width 0.1)
-				(type solid)
-			)
-			(fill no)
-			(layer "F.SilkS")
-		)
 		(fp_circle
 			(center 1.73 -1.73)
@@
 			(layer "F.Fab")
 		)
-		(fp_circle
-			(center 0 0)
-			(end 0.42 0)
-			(stroke
-				(width 0.1)
-				(type solid)
-			)
-			(fill no)
-			(layer "F.Fab")
-		)
 		(fp_text user "${REFERENCE}"
-			(at 0 0 90)
+			(at 0 0 0)
 			(unlocked yes)
 			(layer "F.Fab")
@@
 		)
 		(pad "1" thru_hole circle
-			(at 0 0 90)
+			(at 0 0)
 			(size 2.7 2.7)
 			(drill 1.869999)
 			(layers "*.Cu" "*.Mask")
 			(remove_unused_layers no)
-			(net 4 "/20V_Power_Line/Vin")
+			(net 11 "/20V_Power_Line/Vout")
 			(pinfunction "1")
 			(pintype "unspecified")
@@
 	(footprint "PCM_SL_Mechanical:MountingHole_3.2mm_Pad"
 		(layer "F.Cu")
-		(at 164.5 111.8 180)
+		(at 169.2 111.9 180)
 		(property "Reference" "H1"
 			(at 0 -4.064 180)
@@
 			)
 		)
-		(property "Value" "100p"
+		(property "Value" "110p"
 			(at 0 -4 90)
 			(unlocked yes)
@@
 			)
 		)
-		(property "Datasheet" "https://lcsc.com/product-detail/Multilayer-Ceramic-Capacitors-MLCC-SMD-SMT_100pF-101-5-50V_C1546.html"
+		(property "Datasheet" ""
 			(at 0 0 90)
 			(unlocked yes)
@@
 			)
 		)
-		(property "LCSC Part" "C1546"
+		(property "LCSC Part" "C185562"
 			(at 0 0 90)
 			(unlocked yes)
@@
 			(net 3 "Net-(U4-COMP)")
 			(pinfunction "1")
-			(pintype "input")
+			(pintype "unspecified")
 		)
 		(pad "2" smd rect
@@
 			(net 5 "Net-(U4-FB)")
 			(pinfunction "2")
-			(pintype "input")
+			(pintype "unspecified")
 		)
 		(embedded_fonts no)
@@
 			)
 		)
-		(property "Value" "39n"
+		(property "Value" "150n"
 			(at 0 -4 180)
 			(unlocked yes)
@@
 			)
 		)
-		(property "Datasheet" "https://lcsc.com/product-detail/Multilayer-Ceramic-Capacitors-MLCC-SMD-SMT_39nF-393-10-50V_C1619.html"
+		(property "Datasheet" "https://lcsc.com/product-detail/Multilayer-Ceramic-Capacitors-MLCC-SMD-SMT_150nF-154-10-50V_C1597.html"
 			(at 0 0 180)
 			(unlocked yes)
@@
 			)
 		)
-		(property "LCSC Part" "C1619"
+		(property "LCSC Part" "C1597"
 			(at 0 0 180)
 			(unlocked yes)
